File: Hardware /touch_pot.sch (EAGLE design)
At the start: 72 parts, among them CON1 SINGLE_PADSMD, CON10 SINGLE_PADSMD, CON11 SINGLE_PADSMD, CON12 SINGLE_PADSMD, CON13 SINGLE_PADSMD, CON14 SINGLE_PADSMD, CON15 SINGLE_PADSMD, CON16 SINGLE_PADSMD_R, CON17 SINGLE_PADSMD_R, CON18 SINGLE_PADSMD_R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

Commit message: First Round of changes before Protos
Changed Dimension thickness
Changed silk ratio
Added designed by name
Bumped via size up to 0.020
Added actual stand-offs instead of drill hits
Labeled push button
Parts:
- added STANDOFF1, STANDOFF2: STAND-OFFTIGHT, SparkFun-Electromechanical:STAND-OFFTIGHT
Other:
- note added: "10"
- note removed: "01"
Changed lines of the file:
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@@
 <layer number="54" name="bGND_GNDA" color="1" fill="9" visible="no" active="no"/>
 <layer number="56" name="wert" color="7" fill="1" visible="no" active="no"/>
+<layer number="57" name="tCAD" color="7" fill="1" visible="no" active="no"/>
 <layer number="91" name="Nets" color="2" fill="1" visible="yes" active="yes"/>
 <layer number="92" name="Busses" color="1" fill="1" visible="yes" active="yes"/>
@@
 <layer number="97" name="Info" color="7" fill="1" visible="yes" active="yes"/>
 <layer number="98" name="Guide" color="6" fill="1" visible="yes" active="yes"/>
+<layer number="99" name="SpiceOrder" color="7" fill="1" visible="yes" active="yes"/>
 <layer number="100" name="Muster" color="7" fill="1" visible="no" active="no"/>
 <layer number="101" name="Patch_Top" color="12" fill="4" visible="yes" active="yes"/>
@@
 <layer number="110" name="fp0" color="7" fill="1" visible="no" active="yes"/>
 <layer number="111" name="LPC17xx" color="7" fill="1" visible="yes" active="yes"/>
+<layer number="112" name="tSilk" color="7" fill="1" visible="yes" active="yes"/>
 <layer number="116" name="Patch_BOT" color="9" fill="4" visible="yes" active="yes"/>
 <layer number="121" name="_tsilk" color="7" fill="1" visible="yes" active="yes"/>
@@
 <layer number="124" name="bTestmark" color="7" fill="1" visible="no" active="yes"/>
 <layer number="125" name="_tNames" color="7" fill="1" visible="yes" active="yes"/>
+<layer number="126" name="_bNames" color="7" fill="1" visible="yes" active="yes"/>
+<layer number="127" name="_tValues" color="7" fill="1" visible="yes" active="yes"/>
+<layer number="128" name="_bValues" color="7" fill="1" visible="yes" active="yes"/>
 <layer number="131" name="tAdjust" color="7" fill="1" visible="no" active="yes"/>
 <layer number="132" name="bAdjust" color="7" fill="1" visible="no" active="yes"/>
 <layer number="144" name="Drill_legend" color="7" fill="1" visible="yes" active="yes"/>
+<layer number="150" name="Notes" color="7" fill="1" visible="yes" active="yes"/>
 <layer number="151" name="HeatSink" color="7" fill="1" visible="yes" active="yes"/>
+<layer number="152" name="_bDocu" color="7" fill="1" visible="yes" active="yes"/>
+<layer number="153" name="FabDoc1" color="7" fill="1" visible="yes" active="yes"/>
+<layer number="154" name="FabDoc2" color="7" fill="1" visible="yes" active="yes"/>
+<layer number="155" name="FabDoc3" color="7" fill="1" visible="yes" active="yes"/>
 <layer number="199" name="Contour" color="7" fill="1" visible="yes" active="yes"/>
 <layer number="200" name="200bmp" color="1" fill="10" visible="no" active="no"/>
@@
 <layer number="223" name="223bmp" color="24" fill="1" visible="no" active="no"/>
 <layer number="224" name="224bmp" color="25" fill="1" visible="no" active="no"/>
+<layer number="248" name="Housing" color="7" fill="1" visible="yes" active="yes"/>
+<layer number="249" name="Edge" color="7" fill="1" visible="yes" active="yes"/>
 <layer number="250" name="Descript" color="3" fill="1" visible="no" active="no"/>
 <layer number="251" name="SMDround" color="12" fill="11" visible="no" active="no"/>
@@
 <part name="U$4" library="SparkFun" deviceset="OSHW-LOGO" device="M"/>
 <part name="FRAME3" library="SparkFun-Aesthetics" deviceset="FRAME-LEDGER" device=""/>
+<part name="STANDOFF1" library="SparkFun-Electromechanical" deviceset="STAND-OFF" device="TIGHT"/>
+<part name="STANDOFF2" library="SparkFun-Electromechanical" deviceset="STAND-OFF" device="TIGHT"/>
 </parts>
 <sheets>
@@
 <wire x1="142.24" y1="154.94" x2="142.24" y2="203.2" width="0.1524" layer="97"/>
 <wire x1="185.42" y1="154.94" x2="185.42" y2="203.2" width="0.1524" layer="97"/>
-<text x="355.6" y="10.16" size="2.54" layer="94">danjuliodesigns, LLC</text>
-<text x="421.64" y="7.62" size="2.54" layer="94">01</text>
+<text x="354.838" y="11.43" size="2.54" layer="94">danjuliodesigns, LLC</text>
+<text x="421.64" y="7.62" size="2.54" layer="94">10</text>
 <text x="149.86" y="142.24" size="1.778" layer="97">I2C Address Select</text>
 <text x="86.36" y="261.62" size="1.778" layer="97">IO Connections</text>
@@
 <instance part="FRAME3" gate="G$1" x="0" y="0"/>
 <instance part="FRAME3" gate="G$2" x="330.2" y="0"/>
+<instance part="STANDOFF1" gate="G$1" x="304.8" y="40.64"/>
+<instance part="STANDOFF2" gate="G$1" x="312.42" y="40.64"/>
 </instances>
 <busses>

Commit message: Work in progress
rerouting for fourth standoff hole
Parts:
- added STANDOFF3, STANDOFF4: STAND-OFFTIGHT, SparkFun-Electromechanical:STAND-OFFTIGHT
- added U$5: FIDUCIAL, djd_eagle_library:FIDUCIAL
Changed lines of the file:
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@@
 <?xml version="1.0" encoding="utf-8"?>
 <!DOCTYPE eagle SYSTEM "eagle.dtd">
-<eagle version="6.5.0">
+<eagle version="7.1.0">
 <drawing>
 <settings>
@@
 <part name="U$4" library="SparkFun" deviceset="OSHW-LOGO" device="M"/>
 <part name="FRAME3" library="SparkFun-Aesthetics" deviceset="FRAME-LEDGER" device=""/>
+<part name="STANDOFF3" library="SparkFun-Electromechanical" deviceset="STAND-OFF" device="TIGHT"/>
+<part name="STANDOFF2" library="SparkFun-Electromechanical" deviceset="STAND-OFF" device="TIGHT"/>
+<part name="U$5" library="djd_eagle_library" deviceset="FIDUCIAL" device=""/>
+<part name="STANDOFF4" library="SparkFun-Electromechanical" deviceset="STAND-OFF" device="TIGHT"/>
 <part name="STANDOFF1" library="SparkFun-Electromechanical" deviceset="STAND-OFF" device="TIGHT"/>
-<part name="STANDOFF2" library="SparkFun-Electromechanical" deviceset="STAND-OFF" device="TIGHT"/>
 </parts>
 <sheets>
@@
 <instance part="FRAME3" gate="G$1" x="0" y="0"/>
 <instance part="FRAME3" gate="G$2" x="330.2" y="0"/>
-<instance part="STANDOFF1" gate="G$1" x="304.8" y="40.64"/>
-<instance part="STANDOFF2" gate="G$1" x="312.42" y="40.64"/>
+<instance part="STANDOFF3" gate="G$1" x="312.42" y="40.64"/>
+<instance part="STANDOFF2" gate="G$1" x="320.04" y="40.64"/>
+<instance part="U$5" gate="G$1" x="297.18" y="30.48"/>
+<instance part="STANDOFF4" gate="G$1" x="304.8" y="40.64"/>
+<instance part="STANDOFF1" gate="G$1" x="297.18" y="40.64"/>
 </instances>
 <busses>
