File: Hardware/touch_pot.sch (EAGLE design)
At the start: 78 parts, among them CON1 SINGLE_PADSMD, CON10 SINGLE_PADSMD, CON11 SINGLE_PADSMD, CON12 SINGLE_PADSMD, CON13 SINGLE_PADSMD, CON14 SINGLE_PADSMD, CON15 SINGLE_PADSMD, CON2 SINGLE_PADSMD, CON3 SINGLE_PADSMD, CON4 SINGLE_PADSMD, CON5 SINGLE_PADSMD, CON6 SINGLE_PADSMD, CON7 SINGLE_PADSMD, CON8 SINGLE_PADSMD, CON9 SINGLE_PADSMD, U1 PIC16F1829, U2 AD5262, U3 5V

Commit message: V13
v13
Other:
- note added: "V13"
- note removed: "12"
Changed lines of the file:
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@@
 <wire x1="347.98" y1="226.06" x2="347.98" y2="274.32" width="0.1524" layer="97"/>
 <text x="354.838" y="11.43" size="2.54" layer="94">danjuliodesigns, LLC</text>
-<text x="421.64" y="7.62" size="2.54" layer="94">12</text>
+<text x="421.64" y="7.62" size="2.54" layer="94">V13</text>
 <text x="93.98" y="132.715" size="2.54" layer="97">I2C Address Select</text>
 <text x="22.86" y="264.16" size="2.54" layer="97">IO Connections</text>

Commit message: Clean-up, change button text
Moved traces away from hole, deleted unused ground traces, resized one
trace, changed button text for both i2c and cal.
Other:
- note added: "3 presses - Set I2C Address 4 presses - Start Cal procedure"
- note removed: "I2C Address Select"
Changed lines of the file:
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@@
 <text x="354.838" y="11.43" size="2.54" layer="94">danjuliodesigns, LLC</text>
 <text x="421.64" y="7.62" size="2.54" layer="94">V13</text>
-<text x="93.98" y="132.715" size="2.54" layer="97">I2C Address Select</text>
+<text x="81.28" y="132.715" size="2.54" layer="97">3 presses - Set I2C Address
+4 presses - Start Cal procedure</text>
 <text x="22.86" y="264.16" size="2.54" layer="97">IO Connections</text>
 <text x="218.44" y="274.32" size="2.54" layer="97">ICSP</text>

Commit message: Last QC Check changes
Minor changes based on QC Checklist.
Parts:
- renumbered CON1 to TP6, CON10 to TP15, CON11 to TP16, CON12 to TP17, CON13 to TP18, CON14 to TP19, CON15 to TP20, CON2 to TP7, CON3 to TP8, CON4 to TP9, CON5 to TP10, CON6 to TP11, CON7 to TP12, CON8 to TP13, CON9 to TP14
Other:
- moved on the sheet: C5, C6, C7, C8
